File: tic12400.brd (EAGLE design)
At the start: 100 x 80 mm, 68 parts, among them Q1 CSTCR6M00G53Z, T1_GND gnd, T2_GND gnd, T2_GND1 gnd, U1 TIC12400DCPR, U2 MCZ33996EK, U3 MCP2210-I/SO, U4 BMX160, U5 ON_SEMICONDUCTOR_NCP1117DT33G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, X1 22-23-2031, X2 INPUT1, X3 INPUT2, X4 INPUT3, X5 22-23-2031, X6 OUTPUT1, X7 OUTPUT2, X8 MINI-USB-32005-201

Commit message: up
Parts:
- added USB_D+: d+, wirepad:1,6/0,8
- added USB_D-: d-, wirepad:1,6/0,8
- IMU_INT1: value WIREPAD1,6/0,8 -> int1
- IMU_INT2: value WIREPAD1,6/0,8 -> int2
- renumbered PAD1 to IMU_INT2, PAD2 to IMU_INT1
Connections:
- net N$55: now also USB_D+.1
- net N$56: now also USB_D-.1
Routing:
- net N$55: track 18.1 -> 42.3 mm
- net N$56: track 15.8 -> 31.6 mm
Changed lines of the file:
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@@
 <attribute name="MF" value="NXP USA" x="22.86" y="27.94" size="1.778" layer="27" display="off"/>
 <attribute name="MP" value="MCZ33996EK" x="22.86" y="27.94" size="1.778" layer="27" display="off"/>
+<attribute name="NAME" x="19.459590625" y="34.24075" size="1.27015" layer="25"/>
 <attribute name="NAME" x="19.455309375" y="34.248690625" size="1.27175" layer="25"/>
-<attribute name="NAME" x="19.459590625" y="34.24075" size="1.27015" layer="25"/>
 <attribute name="PACKAGE" value="SOIC-32 NXP Semiconductors" x="22.86" y="27.94" size="1.778" layer="27" display="off"/>
 <attribute name="PRICE" value="None" x="22.86" y="27.94" size="1.778" layer="27" display="off"/>
@@
 <attribute name="VALUE" x="69.85" y="5.08" size="1.27" layer="27" rot="R270"/>
 </element>
-<element name="PAD1" library="wirepad" library_urn="urn:adsk.eagle:library:412" package="1,6/0,8" package3d_urn="urn:adsk.eagle:package:30830/1" value="WIREPAD1,6/0,8" x="74.93" y="6.35" smashed="yes">
+<element name="IMU_INT2" library="wirepad" library_urn="urn:adsk.eagle:library:412" package="1,6/0,8" package3d_urn="urn:adsk.eagle:package:30830/1" value="int2" x="74.93" y="6.35" smashed="yes">
 <attribute name="NAME" x="74.168" y="7.366" size="1.27" layer="25" ratio="10"/>
 <attribute name="POPULARITY" value="1" x="74.93" y="6.35" size="1.778" layer="27" display="off"/>
 <attribute name="VALUE" x="74.93" y="6.95" size="0.0254" layer="27"/>
 </element>
-<element name="PAD2" library="wirepad" library_urn="urn:adsk.eagle:library:412" package="1,6/0,8" package3d_urn="urn:adsk.eagle:package:30830/1" value="WIREPAD1,6/0,8" x="31.75" y="2.54" smashed="yes">
+<element name="IMU_INT1" library="wirepad" library_urn="urn:adsk.eagle:library:412" package="1,6/0,8" package3d_urn="urn:adsk.eagle:package:30830/1" value="int1" x="31.75" y="2.54" smashed="yes">
 <attribute name="NAME" x="30.988" y="3.556" size="1.27" layer="25" ratio="10"/>
 <attribute name="POPULARITY" value="1" x="31.75" y="2.54" size="1.778" layer="27" display="off"/>
@@
 <attribute name="TP_SIGNAL_NAME" value="" x="97.79" y="39.37" size="1.778" layer="27" display="off"/>
 <attribute name="VALUE" x="97.155" y="38.608" size="0.0254" layer="27"/>
+</element>
+<element name="USB_D+" library="wirepad" library_urn="urn:adsk.eagle:library:412" package="1,6/0,8" package3d_urn="urn:adsk.eagle:package:30830/1" value="d+" x="93.98" y="7.62" smashed="yes">
+<attribute name="NAME" x="93.218" y="8.636" size="1.27" layer="25" ratio="10"/>
+<attribute name="POPULARITY" value="1" x="93.98" y="7.62" size="1.778" layer="27" display="off"/>
+<attribute name="VALUE" x="93.98" y="8.22" size="0.0254" layer="27"/>
+</element>
+<element name="USB_D-" library="wirepad" library_urn="urn:adsk.eagle:library:412" package="1,6/0,8" package3d_urn="urn:adsk.eagle:package:30830/1" value="d-" x="93.98" y="2.54" smashed="yes">
+<attribute name="NAME" x="93.218" y="3.556" size="1.27" layer="25" ratio="10"/>
+<attribute name="POPULARITY" value="1" x="93.98" y="2.54" size="1.778" layer="27" display="off"/>
+<attribute name="VALUE" x="93.98" y="3.14" size="0.0254" layer="27"/>
 </element>
 </elements>
@@
 <contactref element="X8" pad="3"/>
 <wire x1="88.2396" y1="21.2598" x2="87.3252" y2="21.2598" width="0.1524" layer="1"/>
-<wire x1="89.154" y1="20.3454" x2="88.2396" y2="21.2598" width="0.1524" layer="1"/>
+<wire x1="89.154" y1="20.3454" x2="88.5825" y2="20.9169" width="0.1524" layer="1"/>
+<wire x1="88.5825" y1="20.9169" x2="88.2396" y2="21.2598" width="0.1524" layer="1"/>
 <wire x1="89.154" y1="18.669" x2="89.154" y2="20.3454" width="0.1524" layer="1"/>
 <wire x1="89.4588" y1="18.3642" x2="89.154" y2="18.669" width="0.1524" layer="1"/>
@@
 <wire x1="87.3252" y1="21.2598" x2="87.325" y2="21.325" width="0.1524" layer="1"/>
 <wire x1="81.3054" y1="9.3726" x2="81.28" y2="9.35" width="0.1524" layer="1"/>
+<contactref element="USB_D+" pad="1"/>
+<wire x1="90.6018" y1="7.62" x2="93.98" y2="7.62" width="0.1524" layer="1"/>
+<wire x1="90.2208" y1="8.001" x2="90.6018" y2="7.62" width="0.1524" layer="1"/>
+<wire x1="90.2208" y1="16.383" x2="90.2208" y2="8.001" width="0.1524" layer="1"/>
+<wire x1="93.726" y1="19.8882" x2="90.2208" y2="16.383" width="0.1524" layer="1"/>
+<wire x1="93.726" y1="21.4122" x2="93.726" y2="19.8882" width="0.1524" layer="1"/>
+<wire x1="93.5736" y1="21.5646" x2="93.726" y2="21.4122" width="0.1524" layer="1"/>
+<wire x1="89.2302" y1="21.5646" x2="93.5736" y2="21.5646" width="0.1524" layer="1"/>
+<wire x1="88.5825" y1="20.9169" x2="89.2302" y2="21.5646" width="0.1524" layer="1"/>
 </signal>
 <signal name="N$56">
@@
 <via x="84.582" y="20.6502" extent="1-16" drill="0.35"/>
 <via x="83.3628" y="13.9446" extent="1-16" drill="0.35"/>
+<contactref element="USB_D-" pad="1"/>
+<wire x1="93.9546" y1="2.8194" x2="93.9546" y2="2.5908" width="0.1524" layer="15"/>
+<wire x1="83.9724" y1="12.8016" x2="93.9546" y2="2.8194" width="0.1524" layer="15"/>
+<wire x1="83.9724" y1="13.335" x2="83.9724" y2="12.8016" width="0.1524" layer="15"/>
+<wire x1="83.3628" y1="13.9446" x2="83.9724" y2="13.335" width="0.1524" layer="15"/>
+<wire x1="93.9546" y1="2.5908" x2="93.98" y2="2.54" width="0.1524" layer="15"/>
 </signal>
 <signal name="N$53">
@@
 <signal name="N$71">
 <contactref element="U4" pad="9"/>
-<contactref element="PAD1" pad="1"/>
+<contactref element="IMU_INT2" pad="1"/>
 <wire x1="70.6374" y1="4.8768" x2="67.2084" y2="4.8768" width="0.1524" layer="1"/>
 <wire x1="72.0852" y1="6.3246" x2="70.6374" y2="4.8768" width="0.1524" layer="1"/>
@@
 <signal name="N$70">
 <contactref element="U4" pad="4"/>
-<contactref element="PAD2" pad="1"/>
+<contactref element="IMU_INT1" pad="1"/>
 <wire x1="62.3316" y1="4.2672" x2="64.8462" y2="4.2672" width="0.1524" layer="1"/>
 <wire x1="60.1218" y1="2.0574" x2="62.3316" y2="4.2672" width="0.1524" layer="1"/>
